File: VGA_breakout/VGA_breakout.sch (KiCad schematic (older format))
At the start: 6 parts, among them J1 Breadboard connector, J2 VGA Port, J3 Holder2, J4 Holder1

Commit message: Small changes, generated gerber files
Parts:
- renumbered J2 to J1, J1 to J2
Changed lines of the file:
@@
 $EndDescr
 $Comp
-L Connector:DB15_Female_HighDensity_MountingHoles J2
+L Connector:DB15_Female_HighDensity_MountingHoles J1
 U 1 1 5FBDA24B
 P 9000 2950
-F 0 "J2" H 9000 3817 50  0000 C CNN
+F 0 "J1" H 9000 3817 50  0000 C CNN
 F 1 "VGA Port" H 9000 3726 50  0000 C CNN
 F 2 "Connector_Dsub:DSUB-15-HD_Female_Horizontal_P2.29x1.98mm_EdgePinOffset8.35mm_Housed_MountingHolesOffset10.89mm" H 8050 3350 50  0001 C CNN
@@
 $EndComp
 $Comp
-L Connector_Generic:Conn_01x15 J1
+L Connector_Generic:Conn_01x15 J2
 U 1 1 5FBDD311
 P 7550 3050
-F 0 "J1" H 7468 3967 50  0000 C CNN
+F 0 "J2" H 7468 3967 50  0000 C CNN
 F 1 "Breadboard connector" H 7468 3876 50  0000 C CNN
 F 2 "Connector_PinHeader_2.54mm:PinHeader_1x15_P2.54mm_Vertical" H 7550 3050 50  0001 C CNN

Commit message: Corrected VGA breakout board DSUB-15 footprint
Parts:
- J1: footprint Connector_Dsub:DSUB-15-HD_Female_Horizontal_P2.29x1.98mm_EdgePinOffset8.35mm_Housed_MountingHolesOffset10.89mm -> VGA_breakout:ICD15S13E4GV00LF; symbol Connector:DB15_Female_HighDensity_MountingHoles -> Connector:DB15_Female_HighDensity
Connections:
- no-connect marks 5 -> 4
Changed lines of the file:
@@
 $EndDescr
 $Comp
-L Connector:DB15_Female_HighDensity_MountingHoles J1
+L Connector:DB15_Female_HighDensity J1
 U 1 1 5FBDA24B
 P 9000 2950
 F 0 "J1" H 9000 3817 50  0000 C CNN
 F 1 "VGA Port" H 9000 3726 50  0000 C CNN
-F 2 "Connector_Dsub:DSUB-15-HD_Female_Horizontal_P2.29x1.98mm_EdgePinOffset8.35mm_Housed_MountingHolesOffset10.89mm" H 8050 3350 50  0001 C CNN
+F 2 "VGA_breakout:ICD15S13E4GV00LF" H 8050 3350 50  0001 C CNN
 F 3 " ~" H 8050 3350 50  0001 C CNN
 	1    9000 2950
@@
 Wire Wire Line
 	9800 2550 9300 2550
-NoConn ~ 9000 3650
 $Comp
 L Connector_Generic:Conn_01x02 J3
