File: UPDI_programmer/UPDI_programmer.sch (KiCad schematic (older format))
At the start: 12 parts

Commit message: Finalized schematic
Parts:
- removed R? (x2): 4K7, symbol Device:R_Small
- added C10: 4,7uF, symbol Device:CP
- added C11, C9: 100nF, symbol Device:C_Small
- added C6: 10nF, symbol Device:C_Small
- added C7, C8: 47pF, symbol Device:C_Small
- added D1: TX, symbol Device:LED
- added D2: RX, symbol Device:LED
- added D3: PWR, symbol Device:LED
- added FB1: FBS, symbol Device:Ferrite_Bead_Small
- added J3: USB_A, symbol Connector:USB_A
- added R1, R4: 4K7, symbol Device:R
- added R2, R3: 27, symbol Device:R
- added R5, R6, R7: 470, symbol Device:R
- added U2: FT230XS, Package_SO:SSOP-16_5.3x6.2mm_P0.65mm, symbol 6502:FT230XS
- gave numbers to parts that had none: 10
Connections:
- net GND: now also C10.2, C11.1, C6.2, C7.2, C8.2, C9.1, D3.1 (K), J3.4 (GND), U2.13 (GND), U2.5 (GND), U2.6 (~CTS)
- net RxD: now also U2.1 (TXD)
- net TxD: now also U2.4 (RXD)
- net UPDI: now also R1.1
- net VCC: now also C10.1, C9.2, FB1.1, R4.1, R6.2, U2.12 (VCC)
- net ~RESET: now also R4.2
- net at J1.1 (DATA), JP1.1: now also R1.2
- new net: C11.2, R5.1, R7.1, U2.10 (3V3OUT), U2.11 (~RES), U2.3 (VCCIO)
- new net: C6.1, FB1.2, J3.1 (VBUS)
- new net: C8.1, J3.2 (D-), R3.2
- new net: C7.1, J3.3 (D+), R2.2
- new net: D1.2 (A), R5.2
- new net: D2.2 (A), R7.2
- new net: D3.2 (A), R6.1
- new net USBD+: R2.1, U2.8 (USBD+)
- new net USBD-: R3.1, U2.9 (USBD-)
- new net ~RXLED: D1.1 (K), U2.14 (CBUS1)
- new net ~TXLED: D2.1 (K), U2.7 (CBUS2)
- no-connect marks 16 -> 20
Other:
- moved on the sheet: JP1

Commit message: First PCB draft
Parts:
- C1, C11, C2, C3, C4, C5, C6, C7, C8, C9: footprint (none) -> Capacitor_SMD:C_1206_3216Metric_Pad1.33x1.80mm_HandSolder
- C10: footprint (none) -> Capacitor_THT:CP_Radial_D4.0mm_P2.00mm
- D1, D2, D3: footprint (none) -> LED_SMD:LED_1206_3216Metric_Pad1.42x1.75mm_HandSolder
- FB1, R1, R2, R3, R4, R5, R6, R7: footprint (none) -> Resistor_SMD:R_1206_3216Metric_Pad1.30x1.75mm_HandSolder
- J1: footprint (none) -> Connector_IDC:IDC-Header_2x03_P2.54mm_Vertical
- J2: footprint (none) -> Connector_PinHeader_2.54mm:PinHeader_2x03_P2.54mm_Vertical
- J3: footprint (none) -> Connector_USB:USB_A_CONNFLY_DS1095-WNR0
- JP1: footprint (none) -> Connector_PinHeader_2.54mm:PinHeader_1x02_P2.54mm_Vertical
- U2: footprint Package_SO:SSOP-16_5.3x6.2mm_P0.65mm -> Package_SO:SSOP-16_4.4x5.2mm_P0.65mm
- Y1: footprint (none) -> Crystal:Crystal_HC49-U_Vertical
Changed lines of the file:
@@
 F 0 "C3" V 1121 1750 50  0000 C CNN
 F 1 "100nF" V 1212 1750 50  0000 C CNN
-F 2 "" H 1350 1750 50  0001 C CNN
+F 2 "Capacitor_SMD:C_1206_3216Metric_Pad1.33x1.80mm_HandSolder" H 1350 1750 50  0001 C CNN
 F 3 "~" H 1350 1750 50  0001 C CNN
 	1    1350 1750
@@
 F 0 "C1" V 1721 1150 50  0000 C CNN
 F 1 "100nF" V 1812 1150 50  0000 C CNN
-F 2 "" H 1950 1150 50  0001 C CNN
+F 2 "Capacitor_SMD:C_1206_3216Metric_Pad1.33x1.80mm_HandSolder" H 1950 1150 50  0001 C CNN
 F 3 "~" H 1950 1150 50  0001 C CNN
 	1    1950 1150
@@
 F 0 "C2" V 2221 1150 50  0000 C CNN
 F 1 "100nF" V 2312 1150 50  0000 C CNN
-F 2 "" H 2450 1150 50  0001 C CNN
+F 2 "Capacitor_SMD:C_1206_3216Metric_Pad1.33x1.80mm_HandSolder" H 2450 1150 50  0001 C CNN
 F 3 "~" H 2450 1150 50  0001 C CNN
 	1    2450 1150
@@
 F 0 "Y1" V 3204 2488 50  0000 L CNN
 F 1 "16MHz" V 3295 2488 50  0000 L CNN
-F 2 "" H 3250 2400 50  0001 C CNN
+F 2 "Crystal:Crystal_HC49-U_Vertical" H 3250 2400 50  0001 C CNN
 F 3 "~" H 3250 2400 50  0001 C CNN
 	1    3250 2400
@@
 F 0 "C4" V 3521 2200 50  0000 C CNN
 F 1 "22pF" V 3612 2200 50  0000 C CNN
-F 2 "" H 3750 2200 50  0001 C CNN
+F 2 "Capacitor_SMD:C_1206_3216Metric_Pad1.33x1.80mm_HandSolder" H 3750 2200 50  0001 C CNN
 F 3 "~" H 3750 2200 50  0001 C CNN
 	1    3750 2200
@@
 F 0 "C5" V 3979 2600 50  0000 C CNN
 F 1 "22pF" V 3888 2600 50  0000 C CNN
-F 2 "" H 3750 2600 50  0001 C CNN
+F 2 "Capacitor_SMD:C_1206_3216Metric_Pad1.33x1.80mm_HandSolder" H 3750 2600 50  0001 C CNN
 F 3 "~" H 3750 2600 50  0001 C CNN
 	1    3750 2600
@@
 F 0 "J2" H 4771 1646 50  0000 R CNN
 F 1 "ICSP" H 4771 1555 50  0000 R CNN
-F 2 "" V 4850 1600 50  0001 C CNN
+F 2 "Connector_PinHeader_2.54mm:PinHeader_2x03_P2.54mm_Vertical" V 4850 1600 50  0001 C CNN
 F 3 " ~" H 3825 1000 50  0001 C CNN
 	1    5100 1550
@@
 F 0 "J1" H 6520 1546 50  0000 R CNN
 F 1 "UPDI" H 6520 1455 50  0000 R CNN
-F 2 "" V 6600 1450 50  0001 C CNN
+F 2 "Connector_IDC:IDC-Header_2x03_P2.54mm_Vertical" V 6600 1450 50  0001 C CNN
 F 3 "https://www.microchip.com/webdoc/GUID-9D10622A-5C16-4405-B092-1BDD437B4976/index.html?GUID-9B349315-2842-4189-B88C-49F4E1055D7F" H 5575 950 50  0001 C CNN
 	1    6850 1500
@@
 F 0 "JP1" H 7700 1312 50  0000 C CNN
 F 1 "UPDI_R4K7" H 7700 1221 50  0000 C CNN
-F 2 "" H 7700 1100 50  0001 C CNN
+F 2 "Connector_PinHeader_2.54mm:PinHeader_1x02_P2.54mm_Vertical" H 7700 1100 50  0001 C CNN
 F 3 "~" H 7700 1100 50  0001 C CNN
 	1    7700 1100
@@
 F 0 "U2" H 6400 4465 50  0000 C CNN
 F 1 "FT230XS" H 6400 4374 50  0000 C CNN
-F 2 "Package_SO:SSOP-16_5.3x6.2mm_P0.65mm" H 6400 4350 50  0001 C CNN
+F 2 "Package_SO:SSOP-16_4.4x5.2mm_P0.65mm" H 6400 4350 50  0001 C CNN
 F 3 "" H 6400 3850 50  0001 C CNN
 	1    6400 3850
@@
 F 0 "J3" H 7807 3217 50  0000 C CNN
 F 1 "USB_A" H 7807 3126 50  0000 C CNN
-F 2 "" H 7900 2700 50  0001 C CNN
+F 2 "Connector_USB:USB_A_CONNFLY_DS1095-WNR0" H 7900 2700 50  0001 C CNN
 F 3 " ~" H 7900 2700 50  0001 C CNN
 	1    7750 2750
@@
 F 0 "FB1" V 8563 2550 50  0000 C CNN
 F 1 "FBS" V 8654 2550 50  0000 C CNN
-F 2 "" V 8730 2550 50  0001 C CNN
+F 2 "Resistor_SMD:R_1206_3216Metric_Pad1.30x1.75mm_HandSolder" V 8730 2550 50  0001 C CNN
 F 3 "~" H 8800 2550 50  0001 C CNN
 	1    8800 2550
@@
 F 0 "C6" H 8242 3096 50  0000 L CNN
 F 1 "10nF" H 8242 3005 50  0000 L CNN
-F 2 "" H 8150 3050 50  0001 C CNN
+F 2 "Capacitor_SMD:C_1206_3216Metric_Pad1.33x1.80mm_HandSolder" H 8150 3050 50  0001 C CNN
 F 3 "~" H 8150 3050 50  0001 C CNN
 	1    8150 3050
@@
 F 0 "C7" H 8642 3096 50  0000 L CNN
 F 1 "47pF" H 8642 3005 50  0000 L CNN
-F 2 "" H 8550 3050 50  0001 C CNN
+F 2 "Capacitor_SMD:C_1206_3216Metric_Pad1.33x1.80mm_HandSolder" H 8550 3050 50  0001 C CNN
 F 3 "~" H 8550 3050 50  0001 C CNN
 	1    8550 3050
@@
 F 0 "C8" H 9042 3096 50  0000 L CNN
 F 1 "47pF" H 9042 3005 50  0000 L CNN
-F 2 "" H 8950 3050 50  0001 C CNN
+F 2 "Capacitor_SMD:C_1206_3216Metric_Pad1.33x1.80mm_HandSolder" H 8950 3050 50  0001 C CNN
 F 3 "~" H 8950 3050 50  0001 C CNN
 	1    8950 3050
@@
 F 0 "R2" V 9300 2750 50  0000 C CNN
 F 1 "27" V 9400 2750 50  0000 C CNN
-F 2 "" V 9330 2750 50  0001 C CNN
+F 2 "Resistor_SMD:R_1206_3216Metric_Pad1.30x1.75mm_HandSolder" V 9330 2750 50  0001 C CNN
 F 3 "~" H 9400 2750 50  0001 C CNN
 	1    9400 2750
@@
 F 0 "R3" V 9500 2850 50  0000 C CNN
 F 1 "27" V 9400 2850 50  0000 C CNN
-F 2 "" V 9330 2850 50  0001 C CNN
+F 2 "Resistor_SMD:R_1206_3216Metric_Pad1.30x1.75mm_HandSolder" V 9330 2850 50  0001 C CNN
 F 3 "~" H 9400 2850 50  0001 C CNN
 	1    9400 2850
@@
 F 0 "R1" V 7600 1400 50  0000 C CNN
 F 1 "4K7" V 7700 1400 50  0000 C CNN
-F 2 "" V 7630 1400 50  0001 C CNN
+F 2 "Resistor_SMD:R_1206_3216Metric_Pad1.30x1.75mm_HandSolder" V 7630 1400 50  0001 C CNN
 F 3 "~" H 7700 1400 50  0001 C CNN
 	1    7700 1400
@@
 F 0 "C9" V 7571 3900 50  0000 C CNN
 F 1 "100nF" V 7662 3900 50  0000 C CNN
-F 2 "" H 7800 3900 50  0001 C CNN
+F 2 "Capacitor_SMD:C_1206_3216Metric_Pad1.33x1.80mm_HandSolder" H 7800 3900 50  0001 C CNN
 F 3 "~" H 7800 3900 50  0001 C CNN
 	1    7800 3900
@@
 F 0 "C11" V 7571 4400 50  0000 C CNN
 F 1 "100nF" V 7662 4400 50  0000 C CNN
-F 2 "" H 7800 4400 50  0001 C CNN
+F 2 "Capacitor_SMD:C_1206_3216Metric_Pad1.33x1.80mm_HandSolder" H 7800 4400 50  0001 C CNN
 F 3 "~" H 7800 4400 50  0001 C CNN
 	1    7800 4400
@@
 F 0 "R5" V 4850 3850 50  0000 C CNN
 F 1 "470" V 4950 3850 50  0000 C CNN
-F 2 "" V 4880 3850 50  0001 C CNN
+F 2 "Resistor_SMD:R_1206_3216Metric_Pad1.30x1.75mm_HandSolder" V 4880 3850 50  0001 C CNN
 F 3 "~" H 4950 3850 50  0001 C CNN
 	1    4950 3850
@@
 F 0 "R7" V 4850 4250 50  0000 C CNN
 F 1 "470" V 4950 4250 50  0000 C CNN
-F 2 "" V 4880 4250 50  0001 C CNN
+F 2 "Resistor_SMD:R_1206_3216Metric_Pad1.30x1.75mm_HandSolder" V 4880 4250 50  0001 C CNN
 F 3 "~" H 4950 4250 50  0001 C CNN
 	1    4950 4250
@@
 F 0 "D1" H 4543 4067 50  0000 C CNN
 F 1 "TX" H 4543 3976 50  0000 C CNN
-F 2 "" H 4550 3850 50  0001 C CNN
+F 2 "LED_SMD:LED_1206_3216Metric_Pad1.42x1.75mm_HandSolder" H 4550 3850 50  0001 C CNN
 F 3 "~" H 4550 3850 50  0001 C CNN
 	1    4550 3850
@@
 F 0 "D2" H 4543 4467 50  0000 C CNN
 F 1 "RX" H 4543 4376 50  0000 C CNN
-F 2 "" H 4550 4250 50  0001 C CNN
+F 2 "LED_SMD:LED_1206_3216Metric_Pad1.42x1.75mm_HandSolder" H 4550 4250 50  0001 C CNN
 F 3 "~" H 4550 4250 50  0001 C CNN
 	1    4550 4250
@@
 F 0 "C10" H 9118 4296 50  0000 L CNN
 F 1 "4,7uF" H 9118 4205 50  0000 L CNN
-F 2 "" H 9038 4100 50  0001 C CNN
+F 2 "Capacitor_THT:CP_Radial_D4.0mm_P2.00mm" H 9038 4100 50  0001 C CNN
 F 3 "~" H 9000 4250 50  0001 C CNN
 	1    9000 4250
@@
 F 0 "R6" V 9250 4000 50  0000 C CNN
 F 1 "470" V 9350 4000 50  0000 C CNN
-F 2 "" V 9280 4000 50  0001 C CNN
+F 2 "Resistor_SMD:R_1206_3216Metric_Pad1.30x1.75mm_HandSolder" V 9280 4000 50  0001 C CNN
 F 3 "~" H 9350 4000 50  0001 C CNN
 	1    9350 4000
@@
 F 0 "D3" V 9639 4132 50  0000 R CNN
 F 1 "PWR" V 9548 4132 50  0000 R CNN
-F 2 "" H 9600 4250 50  0001 C CNN
+F 2 "LED_SMD:LED_1206_3216Metric_Pad1.42x1.75mm_HandSolder" H 9600 4250 50  0001 C CNN
 F 3 "~" H 9600 4250 50  0001 C CNN
 	1    9600 4250
@@
 F 0 "R4" V 3100 3050 50  0000 C CNN
 F 1 "4K7" V 3200 3050 50  0000 C CNN
-F 2 "" V 3130 3050 50  0001 C CNN
+F 2 "Resistor_SMD:R_1206_3216Metric_Pad1.30x1.75mm_HandSolder" V 3130 3050 50  0001 C CNN
 F 3 "~" H 3200 3050 50  0001 C CNN
 	1    3200 3050

Commit message: UPDI PCB RC1
Parts:
- removed J3: USB_A, Connector_USB:USB_A_CONNFLY_DS1095-WNR0, symbol Connector:USB_A
- added J3: USB_B, Connector_USB:USB_B_OST_USB-B1HSxx_Horizontal, symbol Connector:USB_B
- renumbered C8 to C1, C4 to C10, C5 to C11, C7 to C2, C6 to C3, C10 to C4, C1 to C5, C9 to C6, C2 to C7, C3 to C8, C11 to C9, R6 to R1, R3 to R2, R2 to R3, R5 to R4, R7 to R5, R4 to R6, R1 to R7, U2 to U1, U1 to U2
Connections:
- net GND: now also J3.4 (GND)
- net at C3.1, FB1.2: now also J3.1 (VBUS)
- net at C1.1, R2.2: now also J3.2 (D-)
- net at C2.1, R3.2: now also J3.3 (D+)
Changed lines of the file:
@@
 $EndDescr
 $Comp
-L MCU_Microchip_ATmega:ATmega168P-20AU U1
+L MCU_Microchip_ATmega:ATmega168P-20AU U2
 U 1 1 617E7028
 P 2150 2950
-F 0 "U1" H 2150 2900 50  0000 C CNN
+F 0 "U2" H 2150 2900 50  0000 C CNN
 F 1 "ATmega168P-20AU" H 2050 3000 50  0000 C CNN
 F 2 "Package_QFP:TQFP-32_7x7mm_P0.8mm" H 2150 2950 50  0001 C CIN
@@
 	1150 1750 1250 1750
 $Comp
-L Device:C_Small C3
+L Device:C_Small C8
 U 1 1 617ED1FC
 P 1350 1750
-F 0 "C3" V 1121 1750 50  0000 C CNN
+F 0 "C8" V 1121 1750 50  0000 C CNN
 F 1 "100nF" V 1212 1750 50  0000 C CNN
 F 2 "Capacitor_SMD:C_1206_3216Metric_Pad1.33x1.80mm_HandSolder" H 1350 1750 50  0001 C CNN
@@
 NoConn ~ 1550 2050
 $Comp
-L Device:C_Small C1
+L Device:C_Small C5
 U 1 1 617EF17B
 P 1950 1150
-F 0 "C1" V 1721 1150 50  0000 C CNN
+F 0 "C5" V 1721 1150 50  0000 C CNN
 F 1 "100nF" V 1812 1150 50  0000 C CNN
 F 2 "Capacitor_SMD:C_1206_3216Metric_Pad1.33x1.80mm_HandSolder" H 1950 1150 50  0001 C CNN
@@
 $EndComp
 $Comp
-L Device:C_Small C2
+L Device:C_Small C7
 U 1 1 617EF7C0
 P 2450 1150
-F 0 "C2" V 2221 1150 50  0000 C CNN
+F 0 "C7" V 2221 1150 50  0000 C CNN
 F 1 "100nF" V 2312 1150 50  0000 C CNN
 F 2 "Capacitor_SMD:C_1206_3216Metric_Pad1.33x1.80mm_HandSolder" H 2450 1150 50  0001 C CNN
@@
 	3100 2350 2750 2350
 $Comp
-L Device:C_Small C4
+L Device:C_Small C10
 U 1 1 617FAA3A
 P 3750 2200
-F 0 "C4" V 3521 2200 50  0000 C CNN
+F 0 "C10" V 3521 2200 50  0000 C CNN
 F 1 "22pF" V 3612 2200 50  0000 C CNN
 F 2 "Capacitor_SMD:C_1206_3216Metric_Pad1.33x1.80mm_HandSolder" H 3750 2200 50  0001 C CNN
@@
 $EndComp
 $Comp
-L Device:C_Small C5
+L Device:C_Small C11
 U 1 1 617FB085
 P 3750 2600
-F 0 "C5" V 3979 2600 50  0000 C CNN
+F 0 "C11" V 3979 2600 50  0000 C CNN
 F 1 "22pF" V 3888 2600 50  0000 C CNN
 F 2 "Capacitor_SMD:C_1206_3216Metric_Pad1.33x1.80mm_HandSolder" H 3750 2600 50  0001 C CNN
@@
 	8000 1400 8150 1400
 $Comp
-L 6502:FT230XS U2
+L 6502:FT230XS U1
 U 1 1 61806644
 P 6400 3850
-F 0 "U2" H 6400 4465 50  0000 C CNN
+F 0 "U1" H 6400 4465 50  0000 C CNN
 F 1 "FT230XS" H 6400 4374 50  0000 C CNN
 F 2 "Package_SO:SSOP-16_4.4x5.2mm_P0.65mm" H 6400 4350 50  0001 C CNN
 F 3 "" H 6400 3850 50  0001 C CNN
 	1    6400 3850
-	1    0    0    -1
-$EndComp
-$Comp
-L Connector:USB_A J3
-U 1 1 618081BA
-P 7750 2750
-F 0 "J3" H 7807 3217 50  0000 C CNN
-F 1 "USB_A" H 7807 3126 50  0000 C CNN
-F 2 "Connector_USB:USB_A_CONNFLY_DS1095-WNR0" H 7900 2700 50  0001 C CNN
-F 3 " ~" H 7900 2700 50  0001 C CNN
-	1    7750 2750
 	1    0    0    -1
 $EndComp
@@
 	8050 2550 8150 2550
 $Comp
-L Device:C_Small C6
+L Device:C_Small C3
 U 1 1 61812570
 P 8150 3050
-F 0 "C6" H 8242 3096 50  0000 L CNN
+F 0 "C3" H 8242 3096 50  0000 L CNN
 F 1 "10nF" H 8242 3005 50  0000 L CNN
 F 2 "Capacitor_SMD:C_1206_3216Metric_Pad1.33x1.80mm_HandSolder" H 8150 3050 50  0001 C CNN
@@
 	8150 3250 8150 3150
 $Comp
-L Device:C_Small C7
+L Device:C_Small C2
 U 1 1 618178E0
 P 8550 3050
-F 0 "C7" H 8642 3096 50  0000 L CNN
+F 0 "C2" H 8642 3096 50  0000 L CNN
 F 1 "47pF" H 8642 3005 50  0000 L CNN
 F 2 "Capacitor_SMD:C_1206_3216Metric_Pad1.33x1.80mm_HandSolder" H 8550 3050 50  0001 C CNN
@@
 $EndComp
 $Comp
-L Device:C_Small C8
+L Device:C_Small C1
 U 1 1 61817D94
 P 8950 3050
-F 0 "C8" H 9042 3096 50  0000 L CNN
+F 0 "C1" H 9042 3096 50  0000 L CNN
 F 1 "47pF" H 9042 3005 50  0000 L CNN
 F 2 "Capacitor_SMD:C_1206_3216Metric_Pad1.33x1.80mm_HandSolder" H 8950 3050 50  0001 C CNN
@@
 	9550 2850 9650 2850
 $Comp
-L Device:R R2
+L Device:R R3
 U 1 1 61826367
 P 9400 2750
-F 0 "R2" V 9300 2750 50  0000 C CNN
+F 0 "R3" V 9300 2750 50  0000 C CNN
 F 1 "27" V 9400 2750 50  0000 C CNN
 F 2 "Resistor_SMD:R_1206_3216Metric_Pad1.30x1.75mm_HandSolder" V 9330 2750 50  0001 C CNN
@@
 $EndComp
 $Comp
-L Device:R R3
+L Device:R R2
 U 1 1 61828B1F
 P 9400 2850
-F 0 "R3" V 9500 2850 50  0000 C CNN
+F 0 "R2" V 9500 2850 50  0000 C CNN
 F 1 "27" V 9400 2850 50  0000 C CNN
 F 2 "Resistor_SMD:R_1206_3216Metric_Pad1.30x1.75mm_HandSolder" V 9330 2850 50  0001 C CNN
@@
 $EndComp
 $Comp
-L Device:R R1
+L Device:R R7
 U 1 1 6182D165
 P 7700 1400
-F 0 "R1" V 7600 1400 50  0000 C CNN
+F 0 "R7" V 7600 1400 50  0000 C CNN
 F 1 "4K7" V 7700 1400 50  0000 C CNN
 F 2 "Resistor_SMD:R_1206_3216Metric_Pad1.30x1.75mm_HandSolder" V 7630 1400 50  0001 C CNN
@@
 	5700 4100 5850 4100
 $Comp
-L Device:C_Small C9
+L Device:C_Small C6
 U 1 1 61854F3A
 P 7800 3900
-F 0 "C9" V 7571 3900 50  0000 C CNN
+F 0 "C6" V 7571 3900 50  0000 C CNN
 F 1 "100nF" V 7662 3900 50  0000 C CNN
 F 2 "Capacitor_SMD:C_1206_3216Metric_Pad1.33x1.80mm_HandSolder" H 7800 3900 50  0001 C CNN
@@
 	7900 3900 8000 3900
 $Comp
-L Device:C_Small C11
+L Device:C_Small C9
 U 1 1 6185B5B7
 P 7800 4400
-F 0 "C11" V 7571 4400 50  0000 C CNN
+F 0 "C9" V 7571 4400 50  0000 C CNN
 F 1 "100nF" V 7662 4400 50  0000 C CNN
 F 2 "Capacitor_SMD:C_1206_3216Metric_Pad1.33x1.80mm_HandSolder" H 7800 4400 50  0001 C CNN
@@
 	7900 4400 8000 4400
 $Comp
-L Device:R R5
+L Device:R R4
 U 1 1 61863E46
 P 4950 3850
-F 0 "R5" V 4850 3850 50  0000 C CNN
+F 0 "R4" V 4850 3850 50  0000 C CNN
 F 1 "470" V 4950 3850 50  0000 C CNN
 F 2 "Resistor_SMD:R_1206_3216Metric_Pad1.30x1.75mm_HandSolder" V 4880 3850 50  0001 C CNN
@@
 Connection ~ 5200 3850
 $Comp
-L Device:R R7
+L Device:R R5
 U 1 1 618677F6
 P 4950 4250
-F 0 "R7" V 4850 4250 50  0000 C CNN
+F 0 "R5" V 4850 4250 50  0000 C CNN
 F 1 "470" V 4950 4250 50  0000 C CNN
 F 2 "Resistor_SMD:R_1206_3216Metric_Pad1.30x1.75mm_HandSolder" V 4880 4250 50  0001 C CNN
@@
 	4300 3850 4400 3850
 $Comp
-L Device:CP C10
+L Device:CP C4
 U 1 1 61881946
 P 9000 4250
-F 0 "C10" H 9118 4296 50  0000 L CNN
+F 0 "C4" H 9118 4296 50  0000 L CNN
 F 1 "4,7uF" H 9118 4205 50  0000 L CNN
 F 2 "Capacitor_THT:CP_Radial_D4.0mm_P2.00mm" H 9038 4100 50  0001 C CNN
@@
 	9000 4100 9000 4000
 $Comp
-L Device:R R6
+L Device:R R1
 U 1 1 6188F3FB
 P 9350 4000
-F 0 "R6" V 9250 4000 50  0000 C CNN
+F 0 "R1" V 9250 4000 50  0000 C CNN
 F 1 "470" V 9350 4000 50  0000 C CNN
 F 2 "Resistor_SMD:R_1206_3216Metric_Pad1.30x1.75mm_HandSolder" V 9280 4000 50  0001 C CNN
@@
 Connection ~ 2250 1150
 $Comp
-L Device:R R4
+L Device:R R6
 U 1 1 618AC77A
 P 3200 3050
-F 0 "R4" V 3100 3050 50  0000 C CNN
+F 0 "R6" V 3100 3050 50  0000 C CNN
 F 1 "4K7" V 3200 3050 50  0000 C CNN
 F 2 "Resistor_SMD:R_1206_3216Metric_Pad1.30x1.75mm_HandSolder" V 3130 3050 50  0001 C CNN
@@
 Text GLabel 3950 2200 2    50   Output ~ 0
 GND
-$Comp
-L power:VCC #PWR01
-U 1 1 619215B6
-P 9500 2450
-F 0 "#PWR01" H 9500 2300 50  0001 C CNN
-F 1 "VCC" H 9515 2623 50  0000 C CNN
-F 2 "" H 9500 2450 50  0001 C CNN
-F 3 "" H 9500 2450 50  0001 C CNN
-	1    9500 2450
-	1    0    0    -1
-$EndComp
-Wire Wire Line
-	9500 2450 9500 2550
-Connection ~ 9500 2550
-Wire Wire Line
-	9500 2550 9650 2550
-$Comp
-L power:PWR_FLAG #FLG01
-U 1 1 6192FCD6
-P 8350 2450
-F 0 "#FLG01" H 8350 2525 50  0001 C CNN
-F 1 "PWR_FLAG" H 8350 2623 50  0000 C CNN
-F 2 "" H 8350 2450 50  0001 C CNN
-F 3 "~" H 8350 2450 50  0001 C CNN
-	1    8350 2450
-	1    0    0    -1
-$EndComp
-Wire Wire Line
-	8350 2450 8350 2550
 Wire Wire Line
 	8950 3250 9700 3250
@@
 	1    0    0    -1
 $EndComp
-$Comp
-L power:PWR_FLAG #FLG03
-U 1 1 61935AF8
-P 9000 4600
-F 0 "#FLG03" H 9000 4675 50  0001 C CNN
-F 1 "PWR_FLAG" H 9000 4773 50  0000 C CNN
-F 2 "" H 9000 4600 50  0001 C CNN
-F 3 "~" H 9000 4600 50  0001 C CNN
-	1    9000 4600
-	-1   0    0    1
-$EndComp
-Wire Wire Line
-	9000 4600 9000 4500
 Wire Wire Line
 	9000 3900 9000 4000
-Wire Wire Line
-	8900 2550 9500 2550
-Connection ~ 8350 2550
-Wire Wire Line
-	8350 2550 8700 2550
-Wire Wire Line
-	8150 2550 8350 2550
+$Comp
+L Connector:USB_B J3
+U 1 1 619D417A
+P 7750 2750
+F 0 "J3" H 7807 3217 50  0000 C CNN
+F 1 "USB_B" H 7807 3126 50  0000 C CNN
+F 2 "Connector_USB:USB_B_OST_USB-B1HSxx_Horizontal" H 7900 2700 50  0001 C CNN
+F 3 " ~" H 7900 2700 50  0001 C CNN
+	1    7750 2750
+	1    0    0    -1
+$EndComp
+Wire Wire Line
+	8150 2550 8700 2550
+Wire Wire Line
+	8900 2550 9650 2550
 $EndSCHEMATC

Commit message: Updated VIA params and changed UPDI resistor
Parts:
- JP1: value UPDI_R4K7 -> UPDI_R470
- R7: value 4K7 -> 470
Changed lines of the file:
@@
 P 7700 1100
 F 0 "JP1" H 7700 1312 50  0000 C CNN
-F 1 "UPDI_R4K7" H 7700 1221 50  0000 C CNN
+F 1 "UPDI_R470" H 7700 1221 50  0000 C CNN
 F 2 "Connector_PinHeader_2.54mm:PinHeader_1x02_P2.54mm_Vertical" H 7700 1100 50  0001 C CNN
 F 3 "~" H 7700 1100 50  0001 C CNN
@@
 P 7700 1400
 F 0 "R7" V 7600 1400 50  0000 C CNN
-F 1 "4K7" V 7700 1400 50  0000 C CNN
+F 1 "470" V 7700 1400 50  0000 C CNN
 F 2 "Resistor_SMD:R_1206_3216Metric_Pad1.30x1.75mm_HandSolder" V 7630 1400 50  0001 C CNN
 F 3 "~" H 7700 1400 50  0001 C CNN
