File: AVRUPDI_breakout/AVRUPDI_breakout.kicad_pcb (KiCad board)
At the start: 2 copper layers, 11.4 x 17.8 mm, 2 parts, among them J1 UPDI, J2 3PIN

Commit message: PCB RC2
Other:
- rule pad_to_mask_clearance: 0.051 -> 0
Changed lines of the file:
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@@
     (pad_size 1.524 1.524)
     (pad_drill 0.762)
-    (pad_to_mask_clearance 0.051)
-    (solder_mask_min_width 0.25)
+    (pad_to_mask_clearance 0)
     (aux_axis_origin 0 0)
     (visible_elements 7FFFFFFF)
     (pcbplotparams
-      (layerselection 0x010fc_ffffffff)
+      (layerselection 0x010f0_ffffffff)
       (usegerberextensions true)
       (usegerberattributes false)
@@
       (effects (font (size 1 1) (thickness 0.15)))
     )
+    (fp_line (start 4.35 -1.8) (end -1.8 -1.8) (layer F.CrtYd) (width 0.05))
+    (fp_line (start 4.35 6.85) (end 4.35 -1.8) (layer F.CrtYd) (width 0.05))
+    (fp_line (start -1.8 6.85) (end 4.35 6.85) (layer F.CrtYd) (width 0.05))
+    (fp_line (start -1.8 -1.8) (end -1.8 6.85) (layer F.CrtYd) (width 0.05))
+    (fp_line (start -1.33 -1.33) (end 0 -1.33) (layer F.SilkS) (width 0.12))
+    (fp_line (start -1.33 0) (end -1.33 -1.33) (layer F.SilkS) (width 0.12))
+    (fp_line (start 1.27 -1.33) (end 3.87 -1.33) (layer F.SilkS) (width 0.12))
+    (fp_line (start 1.27 1.27) (end 1.27 -1.33) (layer F.SilkS) (width 0.12))
+    (fp_line (start -1.33 1.27) (end 1.27 1.27) (layer F.SilkS) (width 0.12))
+    (fp_line (start 3.87 -1.33) (end 3.87 6.41) (layer F.SilkS) (width 0.12))
+    (fp_line (start -1.33 1.27) (end -1.33 6.41) (layer F.SilkS) (width 0.12))
+    (fp_line (start -1.33 6.41) (end 3.87 6.41) (layer F.SilkS) (width 0.12))
+    (fp_line (start -1.27 0) (end 0 -1.27) (layer F.Fab) (width 0.1))
+    (fp_line (start -1.27 6.35) (end -1.27 0) (layer F.Fab) (width 0.1))
+    (fp_line (start 3.81 6.35) (end -1.27 6.35) (layer F.Fab) (width 0.1))
+    (fp_line (start 3.81 -1.27) (end 3.81 6.35) (layer F.Fab) (width 0.1))
+    (fp_line (start 0 -1.27) (end 3.81 -1.27) (layer F.Fab) (width 0.1))
     (fp_text user %R (at 1.27 2.54) (layer F.Fab)
       (effects (font (size 1 1) (thickness 0.15)))
     )
-    (fp_line (start 0 -1.27) (end 3.81 -1.27) (layer F.Fab) (width 0.1))
-    (fp_line (start 3.81 -1.27) (end 3.81 6.35) (layer F.Fab) (width 0.1))
-    (fp_line (start 3.81 6.35) (end -1.27 6.35) (layer F.Fab) (width 0.1))
-    (fp_line (start -1.27 6.35) (end -1.27 0) (layer F.Fab) (width 0.1))
-    (fp_line (start -1.27 0) (end 0 -1.27) (layer F.Fab) (width 0.1))
-    (fp_line (start -1.33 6.41) (end 3.87 6.41) (layer F.SilkS) (width 0.12))
-    (fp_line (start -1.33 1.27) (end -1.33 6.41) (layer F.SilkS) (width 0.12))
-    (fp_line (start 3.87 -1.33) (end 3.87 6.41) (layer F.SilkS) (width 0.12))
-    (fp_line (start -1.33 1.27) (end 1.27 1.27) (layer F.SilkS) (width 0.12))
-    (fp_line (start 1.27 1.27) (end 1.27 -1.33) (layer F.SilkS) (width 0.12))
-    (fp_line (start 1.27 -1.33) (end 3.87 -1.33) (layer F.SilkS) (width 0.12))
-    (fp_line (start -1.33 0) (end -1.33 -1.33) (layer F.SilkS) (width 0.12))
-    (fp_line (start -1.33 -1.33) (end 0 -1.33) (layer F.SilkS) (width 0.12))
-    (fp_line (start -1.8 -1.8) (end -1.8 6.85) (layer F.CrtYd) (width 0.05))
-    (fp_line (start -1.8 6.85) (end 4.35 6.85) (layer F.CrtYd) (width 0.05))
-    (fp_line (start 4.35 6.85) (end 4.35 -1.8) (layer F.CrtYd) (width 0.05))
-    (fp_line (start 4.35 -1.8) (end -1.8 -1.8) (layer F.CrtYd) (width 0.05))
     (pad 6 thru_hole oval (at 2.54 5.08 270) (size 1.7 1.7) (drill 1) (layers *.Cu *.Mask)
       (net 4 /GND))
@@
       (effects (font (size 1 1) (thickness 0.15)) (justify mirror))
     )
+    (fp_line (start 1.8 1.8) (end -1.8 1.8) (layer B.CrtYd) (width 0.05))
+    (fp_line (start 1.8 -6.85) (end 1.8 1.8) (layer B.CrtYd) (width 0.05))
+    (fp_line (start -1.8 -6.85) (end 1.8 -6.85) (layer B.CrtYd) (width 0.05))
+    (fp_line (start -1.8 1.8) (end -1.8 -6.85) (layer B.CrtYd) (width 0.05))
+    (fp_line (start -1.33 1.33) (end 0 1.33) (layer B.SilkS) (width 0.12))
+    (fp_line (start -1.33 0) (end -1.33 1.33) (layer B.SilkS) (width 0.12))
+    (fp_line (start -1.33 -1.27) (end 1.33 -1.27) (layer B.SilkS) (width 0.12))
+    (fp_line (start 1.33 -1.27) (end 1.33 -6.41) (layer B.SilkS) (width 0.12))
+    (fp_line (start -1.33 -1.27) (end -1.33 -6.41) (layer B.SilkS) (width 0.12))
+    (fp_line (start -1.33 -6.41) (end 1.33 -6.41) (layer B.SilkS) (width 0.12))
+    (fp_line (start -1.27 0.635) (end -0.635 1.27) (layer B.Fab) (width 0.1))
+    (fp_line (start -1.27 -6.35) (end -1.27 0.635) (layer B.Fab) (width 0.1))
+    (fp_line (start 1.27 -6.35) (end -1.27 -6.35) (layer B.Fab) (width 0.1))
+    (fp_line (start 1.27 1.27) (end 1.27 -6.35) (layer B.Fab) (width 0.1))
     (fp_line (start -0.635 1.27) (end 1.27 1.27) (layer B.Fab) (width 0.1))
-    (fp_line (start 1.27 1.27) (end 1.27 -6.35) (layer B.Fab) (width 0.1))
-    (fp_line (start 1.27 -6.35) (end -1.27 -6.35) (layer B.Fab) (width 0.1))
-    (fp_line (start -1.27 -6.35) (end -1.27 0.635) (layer B.Fab) (width 0.1))
-    (fp_line (start -1.27 0.635) (end -0.635 1.27) (layer B.Fab) (width 0.1))
-    (fp_line (start -1.33 -6.41) (end 1.33 -6.41) (layer B.SilkS) (width 0.12))
-    (fp_line (start -1.33 -1.27) (end -1.33 -6.41) (layer B.SilkS) (width 0.12))
-    (fp_line (start 1.33 -1.27) (end 1.33 -6.41) (layer B.SilkS) (width 0.12))
-    (fp_line (start -1.33 -1.27) (end 1.33 -1.27) (layer B.SilkS) (width 0.12))
-    (fp_line (start -1.33 0) (end -1.33 1.33) (layer B.SilkS) (width 0.12))
-    (fp_line (start -1.33 1.33) (end 0 1.33) (layer B.SilkS) (width 0.12))
-    (fp_line (start -1.8 1.8) (end -1.8 -6.85) (layer B.CrtYd) (width 0.05))
-    (fp_line (start -1.8 -6.85) (end 1.8 -6.85) (layer B.CrtYd) (width 0.05))
-    (fp_line (start 1.8 -6.85) (end 1.8 1.8) (layer B.CrtYd) (width 0.05))
-    (fp_line (start 1.8 1.8) (end -1.8 1.8) (layer B.CrtYd) (width 0.05))
     (fp_text user %R (at 0 -2.54 180) (layer B.Fab)
       (effects (font (size 1 1) (thickness 0.15)) (justify mirror))
